File: kicad/02-S-4r/BlinkySWR-0.2-S.kicad_pcb (KiCad board)
At the start: 2 copper layers, 34.5 x 26.5 mm, 46 parts, among them IC1 ATTINY13A-SSH, J1 SMA-15, J2 SMA-15*, U1 HT7125-1

Commit message: pcb rev0.2
Connections:
- net +3V renamed +2,5V
